File: io.kicad_sch (KiCad schematic)
At the start: 11 parts

Commit message: Added PD chip with footprint, I2C extension connectors
Parts:
- added C? (x2): 100nF 16V, Capacitor_SMD:C_0402_1005Metric, symbol Device:C_Small
- added C?: 10uF 6.3V, Capacitor_SMD:C_0402_1005Metric, symbol Device:C_Small
- added J?: JST_SH_4Pin_Horizontal, MaxTailsLibrary:BOOMELE_SH_1x04_P1.00mm_Horizontal, symbol Connector_Generic:Conn_01x04
- added J?: 01x04 2.54mm, Connector_PinHeader_2.54mm:PinHeader_1x04_P2.54mm_Vertical, symbol Connector_Generic:Conn_01x04
Connections:
- net VDD is gone; now on net +3V3: U?.5 (VDDIO), U?.8 (VDD)
- net +3V3: now also C?.1, C?.1, C?.1, J?.1 (Pin_1), J?.2 (Pin_2)
- net GND: now also C?.2, C?.2, C?.2, J?.1 (Pin_1), J?.4 (Pin_4)
- net CIPO: now reaches U?.1 (SDO/SA0)
- net IMU_CS: now reaches U?.12 (CS)
- net SCK: now reaches U?.13 (SCL)
- net COPI: now reaches U?.14 (SDA)
- new net SCL: J?.3 (Pin_3), J?.4 (Pin_4)
- new net SDA: J?.2 (Pin_2), J?.3 (Pin_3)
Other:
- note added: "(footprint only)"
- note added: "I2C EXT"
- note added: "QWIIC"
- note added: "TODO: - what should be measured - which ESP32 ADC range to choose - maybe external ADC?"
- note removed: "TODO: - what should be measured - which ESP32 ADC range to choose"
- note removed: "TODO: I2C vs SPI"
- moved on the sheet: U?
