File: mcu.kicad_sch (KiCad schematic)
At the start: 0 parts

Commit message: Squashed commit of the following:
commit 867633eb8bb01418950c5f115ec5b264e9701322
Author: CoilProtogen <coilprotogen@gmail.com>
Date:   Tue Jun 28 20:55:42 2022 +0200

    changed naming scheme

commit a153de9a66f35b18339405a8c332f15bc022f5d7
Author: CoilProtogen <coilprotogen@gmail.com>
Date:   Tue Jun 28 20:47:51 2022 +0200

    Added stubs for IO, power, PD

commit 6752e35ff1e8f9ce75f4fd3c7e7d1c6a0aac4c9b
Author: CoilProtogen <coilprotogen@gmail.com>
Date:   Tue Jun 28 00:06:29 2022 +0200

    Initial work on MCU schematic
Parts:
- added AE?: Antenna_Trace, RF_Antenna:Texas_SWRA117D_2.4GHz_Left, symbol Device:Antenna_Shield
- added C? (x5): 100nF 16V, Capacitor_SMD:C_0402_1005Metric, symbol Device:C_Small
- added C?: 10uF 6.3V, Capacitor_SMD:C_0402_1005Metric, symbol Device:C_Small
- added C? (x2): DNP, Capacitor_SMD:C_0402_1005Metric, symbol Device:C_Small
- added J?: 02x05 1.27mm, symbol Connector_Generic:Conn_02x05_Odd_Even
- added Q? (x2): Q_NPN_BEC, Package_TO_SOT_SMD:SOT-23, symbol Device:Q_NPN_BEC
- added R? (x3): 10k, Resistor_SMD:R_0402_1005Metric, symbol Device:R_Small
- added R?: 0R, Resistor_SMD:R_0402_1005Metric, symbol Device:R_Small
- added SW? (x4): SW_Push, Button_Switch_SMD:SW_Push_SPST_NO_Alps_SKRK, symbol Switch:SW_Push
- added U?: ESP32-PICO-V3, Package_DFN_QFN:QFN-48-1EP_7x7mm_P0.5mm_EP5.3x5.3mm, symbol RF_Module:ESP32-PICO-D4
Connections:
- new net: AE?.1 (A), C?.1, R?.2
- new net: C?.1, R?.1, U?.2 (LNA_IN)
- new net: Q?.1 (B), R?.2 (x2)
- new net +3V3: C?.1, C?.1, C?.1, C?.1, C?.1, J?.1 (Pin_1), R?.1, U?.1 (VDDA), U?.19 (VDD3P3_RTC), U?.3 (VDDA3P3), U?.37 (VDD3P3_CPU), U?.4 (VDDA3P3), U?.43 (VDDA), U?.46 (VDDA)
- new net ADC0: U?.5 (SENSOR_VP)
- new net ADC1: U?.6 (SENSOR_CAPP)
- new net ADC2: U?.7 (SENSOR_CAPN)
- new net ADC3: U?.8 (SENSOR_VN)
- new net BUTTON0: SW?.2
- new net BUTTON1: SW?.2
- new net EN: C?.1, Q?.3 (C), R?.2, SW?.2, U?.9 (EN)
- new net ESP_RXD: U?.40 (U0RXD/IO3)
- new net ESP_TXD: U?.41 (U0TXD/IO1)
- new net GND: AE?.2 (Shield), C?.2, C?.2, C?.2, C?.2, C?.2, C?.2, C?.2, C?.2, J?.3 (Pin_3), J?.5 (Pin_5), SW?.1, SW?.1, SW?.1, SW?.1, U?.49 (GND)
- new net IO0: Q?.3 (C), SW?.2, U?.23 (IO0)
- new net MTCK: J?.4 (Pin_4), U?.20 (IO13)
- new net MTDI: J?.8 (Pin_8), U?.18 (IO12)
- new net MTDO: J?.6 (Pin_6), U?.21 (IO15)
- new net MTMS: J?.2 (Pin_2), U?.17 (IO14)
- new net ~{DTR}: Q?.2 (E), R?.1
- new net ~{RTS}: Q?.2 (E), R?.1
- no-connect marks 0 -> 14
Other:
- note added: "ADC max value ~2.45V (4.1.2 esp32 datasheet note)"
- note added: "Compatibility with ESP32PICOD4: avoid using pins: 25, 27, 32, 33, 35, 36"
- note added: "GND Detect pin"
- note added: "JTAG connector"
- note added: "Key pin"
- note added: "RST (Not present)"
- note added: "Strapping pins: EN - high at boot IO0 - high at boot IO2 - low for programming MTDI(IO12) - low at boot MTDO(IO15) - high at boot IO5 - high at boot"
- note added: "TODO: - make ESP footprint conforming to datasheet (inlcuding solder paste/mask) - add testpoints"
- note added: "TODO: Debounce caps?"
- note added: "Truth table: DTR RTS-->EN IO0 1 1 1 1 0 0 1 1 1 0 0 1 0 1 1 0"
- note added: "Use this amplifier? Need docs"

Commit message: Added PD chip with footprint, I2C extension connectors
Parts:
- added R? (x2): 2.2k, Resistor_SMD:R_0402_1005Metric, symbol Device:R_Small
- J?: footprint (none) -> Connector_PinHeader_1.27mm:PinHeader_2x05_P1.27mm_Vertical; now left out of the parts list
Connections:
- net +3V3: now also R?.1, R?.1
- net ADC0: no longer names the net of U?.5 (SENSOR_VP)
- net ADC1: no longer names the net of U?.6 (SENSOR_CAPP)
- net ADC2: no longer names the net of U?.7 (SENSOR_CAPN)
- net ADC3: no longer names the net of U?.8 (SENSOR_VN)
- new net SCL: R?.2
- new net SDA: R?.2
Other:
- note added: "JTAG connector (footprint only)"
- note removed: "JTAG connector"
- note removed: "Use this amplifier? Need docs"
